File: OpenC64Saver.sch (KiCad schematic (older format))
At the start: 17 parts, among them J1 Power I/O, Q1 PN2222A, Q2 PN2222A, X1 OSHW_LOGO, X2 SCREW_HOLE, X3 SCREW_HOLE

Commit message: Experimental full through-hole version
Parts:
- C1: footprint Resistors_SMD:R_0805_HandSoldering -> Capacitor_THT:C_Disc_D7.0mm_W2.5mm_P5.00mm; symbol C -> OpenC64Saver-rescue:C
- D1: symbol D_Zener -> OpenC64Saver-rescue:D_Zener
- D2: symbol D -> OpenC64Saver-rescue:D
- D3: symbol LED_Dual_ACA -> OpenC64Saver-rescue:LED_Dual_ACA
- J1: symbol Screw_Terminal_1x03 -> OpenC64Saver-rescue:Screw_Terminal_1x03
- Q1, Q2: symbol PN2222A -> OpenC64Saver-rescue:PN2222A
- R1, R3, R4, R5, R6: footprint Resistors_SMD:R_0805_HandSoldering -> Resistor_THT:R_Axial_DIN0207_L6.3mm_D2.5mm_P10.16mm_Horizontal; symbol R -> OpenC64Saver-rescue:R
- R2: symbol R_Variable -> OpenC64Saver-rescue:R_Variable
- RL1: symbol SRD-05VDC-SL-C -> OpenC64Saver-rescue:SRD-05VDC-SL-C
- X1, X2, X3: symbol CONN_01X01 -> OpenC64Saver-rescue:CONN_01X01
Changed lines of the file:
@@
-EESchema Schematic File Version 2
-LIBS:power
-LIBS:device
-LIBS:transistors
-LIBS:conn
-LIBS:linear
-LIBS:regul
-LIBS:74xx
-LIBS:cmos4000
-LIBS:adc-dac
-LIBS:memory
-LIBS:xilinx
-LIBS:microcontrollers
-LIBS:dsp
-LIBS:microchip
-LIBS:analog_switches
-LIBS:motorola
-LIBS:texas
-LIBS:intel
-LIBS:audio
-LIBS:interface
-LIBS:digital-audio
-LIBS:philips
-LIBS:display
-LIBS:cypress
-LIBS:siliconi
-LIBS:opto
-LIBS:atmel
-LIBS:contrib
-LIBS:valves
-LIBS:relays
+EESchema Schematic File Version 4
 LIBS:OpenC64Saver-cache
-EELAYER 25 0
+EELAYER 26 0
 EELAYER END
 $Descr A4 11693 8268
@@
 Sheet 1 1
 Title "Open C64 Saver"
-Date "2018-01-04"
-Rev "3"
+Date "2018-09-16"
+Rev "4"
 Comp "SukkoPera"
 Comment1 "Original circuit by Ray Carlsen CET - Carlsen Electronics"
@@
 $EndDescr
 $Comp
-L PN2222A Q2
+L OpenC64Saver-rescue:PN2222A Q2
 U 1 1 59765C85
 P 5250 2600
@@
 $EndComp
 $Comp
-L PN2222A Q1
+L OpenC64Saver-rescue:PN2222A Q1
 U 1 1 59765D89
 P 4500 2900
@@
 $EndComp
 $Comp
-L GND #PWR01
+L OpenC64Saver-rescue:GND #PWR01
 U 1 1 59765E30
 P 4200 3600
@@
 $EndComp
 $Comp
-L R R1
+L OpenC64Saver-rescue:R R1
 U 1 1 59765E4A
 P 4200 2000
 F 0 "R1" V 4280 2000 50  0000 C CNN
 F 1 "820" V 4200 2000 50  0000 C CNN
-F 2 "Resistors_SMD:R_0805_HandSoldering" V 4130 2000 50  0001 C CNN
+F 2 "Resistor_THT:R_Axial_DIN0207_L6.3mm_D2.5mm_P10.16mm_Horizontal" V 4130 2000 50  0001 C CNN
 F 3 "" H 4200 2000 50  0000 C CNN
 	1    4200 2000
@@
 $EndComp
 $Comp
-L D_Zener D1
+L OpenC64Saver-rescue:D_Zener D1
 U 1 1 59765F9C
 P 4200 1550
@@
 $EndComp
 $Comp
-L R R3
+L OpenC64Saver-rescue:R R3
 U 1 1 5976603D
 P 4950 2300
 F 0 "R3" V 5030 2300 50  0000 C CNN
 F 1 "220k" V 4950 2300 50  0000 C CNN
-F 2 "Resistors_SMD:R_0805_HandSoldering" V 4880 2300 50  0001 C CNN
+F 2 "Resistor_THT:R_Axial_DIN0207_L6.3mm_D2.5mm_P10.16mm_Horizontal" V 4880 2300 50  0001 C CNN
 F 3 "" H 4950 2300 50  0000 C CNN
 	1    4950 2300
@@
 $EndComp
 $Comp
-L C C1
+L OpenC64Saver-rescue:C C1
 U 1 1 597660AB
 P 6050 2600
 F 0 "C1" H 6075 2700 50  0000 L CNN
 F 1 "0.2u" H 6075 2500 50  0000 L CNN
-F 2 "Resistors_SMD:R_0805_HandSoldering" H 6088 2450 50  0001 C CNN
+F 2 "Capacitor_THT:C_Disc_D7.0mm_W2.5mm_P5.00mm" H 6088 2450 50  0001 C CNN
 F 3 "" H 6050 2600 50  0000 C CNN
 	1    6050 2600
@@
 $EndComp
 Wire Wire Line
-	4200 2150 4200 3050
+	4200 2150 4200 2300
 Wire Wire Line
 	4200 2900 4300 2900
 Wire Wire Line
-	4200 3350 4200 3600
-Wire Wire Line
-	4200 3500 6600 3500
+	4200 3350 4200 3500
+Wire Wire Line
+	4200 3500 4600 3500
 Wire Wire Line
 	4600 3500 4600 3100
 Connection ~ 4200 2900
 Wire Wire Line
-	4600 1950 4600 2700
+	4600 1950 4600 2600
 Wire Wire Line
 	4600 2600 5050 2600
@@
 Connection ~ 4600 3500
 Wire Wire Line
-	5350 2000 5350 2400
+	5350 2000 5350 2150
 Connection ~ 4200 2300
 Wire Wire Line
-	5100 2300 6050 2300
+	5100 2300 5350 2300
 Wire Wire Line
 	4200 2300 4800 2300
@@
 Connection ~ 5350 3500
 Wire Wire Line
-	5350 1350 5350 1700
-Wire Wire Line
-	4200 1350 6600 1350
+	5350 1350 5350 1550
+Wire Wire Line
+	4200 1350 4600 1350
 Wire Wire Line
 	4200 1350 4200 1400
 $Comp
-L VCC #PWR02
+L OpenC64Saver-rescue:VCC #PWR02
 U 1 1 59766225
 P 4200 1350
@@
 	4200 1700 4200 1850
 $Comp
-L R R4
+L OpenC64Saver-rescue:R R4
 U 1 1 597663FA
 P 4600 1800
 F 0 "R4" V 4680 1800 50  0000 C CNN
 F 1 "2.2k" V 4600 1800 50  0000 C CNN
-F 2 "Resistors_SMD:R_0805_HandSoldering" V 4530 1800 50  0001 C CNN
+F 2 "Resistor_THT:R_Axial_DIN0207_L6.3mm_D2.5mm_P10.16mm_Horizontal" V 4530 1800 50  0001 C CNN
 F 3 "" H 4600 1800 50  0000 C CNN
 	1    4600 1800
@@
 Connection ~ 4600 2600
 $Comp
-L SRD-05VDC-SL-C RL1
+L OpenC64Saver-rescue:SRD-05VDC-SL-C RL1
 U 1 1 59766AA9
 P 6200 1650
@@
 $EndComp
 $Comp
-L D D2
+L OpenC64Saver-rescue:D D2
 U 1 1 59766BE3
 P 5350 1850
@@
 Connection ~ 5350 2150
 $Comp
-L R R5
+L OpenC64Saver-rescue:R R5
 U 1 1 597671B5
 P 6500 2500
 F 0 "R5" V 6580 2500 50  0000 C CNN
 F 1 "1k" V 6500 2500 50  0000 C CNN
-F 2 "Resistors_SMD:R_0805_HandSoldering" V 6430 2500 50  0001 C CNN
+F 2 "Resistor_THT:R_Axial_DIN0207_L6.3mm_D2.5mm_P10.16mm_Horizontal" V 6430 2500 50  0001 C CNN
 F 3 "" H 6500 2500 50  0000 C CNN
 	1    6500 2500
@@
 	6500 2150 6500 2350
 $Comp
-L PWR_FLAG #FLG03
+L OpenC64Saver-rescue:PWR_FLAG #FLG03
 U 1 1 5976759E
 P 10050 1050
@@
 $EndComp
 $Comp
-L +5V #PWR04
+L OpenC64Saver-rescue:+5V #PWR04
 U 1 1 597675D9
 P 7200 2200
@@
 $EndComp
 Wire Wire Line
-	6700 2150 6700 2350
+	6700 2150 6700 2250
 Wire Wire Line
 	6700 2250 7200 2250
@@
 	7200 2250 7200 2200
 $Comp
-L +5V #PWR05
+L OpenC64Saver-rescue:+5V #PWR05
 U 1 1 597677F9
 P 9900 2300
@@
 $EndComp
 $Comp
-L GND #PWR06
+L OpenC64Saver-rescue:GND #PWR06
 U 1 1 59767852
 P 10100 2300
@@
 $EndComp
 $Comp
-L VCC #PWR07
+L OpenC64Saver-rescue:VCC #PWR07
 U 1 1 59767884
 P 9500 2300
@@
 	10100 2000 10100 2300
 $Comp
-L VCC #PWR08
+L OpenC64Saver-rescue:VCC #PWR08
 U 1 1 59767AEF
 P 10050 800
@@
 $EndComp
 $Comp
-L PWR_FLAG #FLG09
+L OpenC64Saver-rescue:PWR_FLAG #FLG09
 U 1 1 59767B39
 P 10500 850
@@
 $EndComp
 $Comp
-L GND #PWR010
+L OpenC64Saver-rescue:GND #PWR010
 U 1 1 59767B6B
 P 10500 1050
@@
 	6600 3500 6600 3350
 $Comp
-L R R6
+L OpenC64Saver-rescue:R R6
 U 1 1 59768A52
 P 6700 2500
 F 0 "R6" V 6780 2500 50  0000 C CNN
 F 1 "1k" V 6700 2500 50  0000 C CNN
-F 2 "Resistors_SMD:R_0805_HandSoldering" V 6630 2500 50  0001 C CNN
+F 2 "Resistor_THT:R_Axial_DIN0207_L6.3mm_D2.5mm_P10.16mm_Horizontal" V 6630 2500 50  0001 C CNN
 F 3 "" H 6700 2500 50  0000 C CNN
 	1    6700 2500
@@
 Connection ~ 5350 1350
 $Comp
-L Screw_Terminal_1x03 J1
+L OpenC64Saver-rescue:Screw_Terminal_1x03 J1
 U 1 1 5976AA96
 P 9700 2600
@@
 $EndComp
 $Comp
-L LED_Dual_ACA D3
+L OpenC64Saver-rescue:LED_Dual_ACA D3
 U 1 1 5976BDA1
 P 6600 3050
@@
 $EndComp
 $Comp
-L +5V #PWR011
+L OpenC64Saver-rescue:+5V #PWR011
 U 1 1 59AAFA20
 P 9600 800
@@
 $EndComp
 $Comp
-L PWR_FLAG #FLG012
+L OpenC64Saver-rescue:PWR_FLAG #FLG012
 U 1 1 59AAFA58
 P 9600 1050
@@
 OUTPUT
 $Comp
-L R_Variable R2
+L OpenC64Saver-rescue:R_Variable R2
 U 1 1 59768CBA
 P 4200 3200
@@
 A different R1 might be needed,\ndepending on the particular\nZener diode used.\nI had to use 2.2k, for instance.
 $Comp
-L CONN_01X01 X2
+L OpenC64Saver-rescue:CONN_01X01 X2
 U 1 1 59D9407F
 P 10400 6300
@@
 $EndComp
 $Comp
-L CONN_01X01 X1
+L OpenC64Saver-rescue:CONN_01X01 X1
 U 1 1 59D9413E
 P 9900 6300
@@
 NoConn ~ 10400 6100
 $Comp
-L CONN_01X01 X3
+L OpenC64Saver-rescue:CONN_01X01 X3
 U 1 1 59D94B0F
 P 10900 6300
@@
 $EndComp
 NoConn ~ 10900 6100
+Wire Wire Line
+	4200 2900 4200 3050
+Wire Wire Line
+	4600 3500 5350 3500
+Wire Wire Line
+	4200 2300 4200 2900
+Wire Wire Line
+	5350 2300 5350 2400
+Wire Wire Line
+	5350 2300 6050 2300
+Wire Wire Line
+	5350 3500 6050 3500
+Wire Wire Line
+	4600 1350 5350 1350
+Wire Wire Line
+	4600 2600 4600 2700
+Wire Wire Line
+	5350 1550 5350 1700
+Wire Wire Line
+	5350 2150 5350 2300
+Wire Wire Line
+	6050 3500 6600 3500
+Wire Wire Line
+	6700 2250 6700 2350
+Wire Wire Line
+	4200 3500 4200 3600
+Wire Wire Line
+	5350 1350 6600 1350
 $EndSCHEMATC
